Commit message: Add arm and build platform to the robot

File: jenga_robot_description/urdf/build_platform.urdf.xacro (robot description, xacro)
@@ -5,11 +5,11 @@
    <xacro:property name="M_PI" value="3.14159"/>
    <xacro:include filename="$(find widowx_arm_description)/urdf/common_materials.xacro" />
-   <xacro:macro name="arm_turntable" params="parent prefix *origin">
+   <xacro:macro name="build_platform" params="parent prefix *origin">
       <!-- links -->
-      <link name="${prefix}turntable_main_link">
+      <link name="${prefix}build_platform_main_link">
          <visual>
             <origin xyz="0 0 0" rpy="0 0 0" />
             <geometry>
-		<cylinder length="${FRAME_SCALE*1.25}" radius="${FRAME_SCALE*9}"/>
+		<box size="${FRAME_SCALE*24} ${FRAME_SCALE*21} ${FRAME_SCALE*0.1}" />
             </geometry>
             <xacro:material_black />
@@ -18,5 +18,5 @@
             <origin xyz="0 0 0" rpy="0 0 0" />
             <geometry>
-		<cylinder length="${FRAME_SCALE*1.25}" radius="${FRAME_SCALE*9}"/>
+		<box size="${FRAME_SCALE*24} ${FRAME_SCALE*21} ${FRAME_SCALE*0.1}" />
             </geometry>
          </collision>
@@ -27,23 +27,9 @@
          </inertial>
       </link>
-      <link name="${prefix}arm_mount_link">
-         <inertial>
-            <origin xyz="0 0 0" rpy="0 0 0" />
-            <mass value="1" />
-            <inertia ixx="1.0" ixy="0.0" ixz="0.0" iyy="1.0" iyz="0.0" izz="1.0" />
-         </inertial>
-      </link>
       <!-- joints -->
-      <joint name="${prefix}turntable_joint" type="revolute">
+      <joint name="${prefix}build_platform_joint" type="fixed">
          <xacro:insert_block name="origin" />
          <parent link="${parent}" />
-         <child link="${prefix}turntable_main_link"/>
-         <axis xyz="0 0 1" />
-         <limit lower="${-M_PI/2}" upper="${M_PI/2}" effort="6" velocity="1.571" />
-      </joint>
-      <joint name="${prefix}arm_mount_joint" type="fixed">
-         <origin xyz="${FRAME_SCALE*4.5} 0 ${FRAME_SCALE*-1.25}" rpy="0 ${M_PI} 0" />
-         <parent link="${prefix}turntable_main_link" />
-         <child link="${prefix}arm_mount_link" />
+         <child link="${prefix}build_platform_main_link"/>
       </joint>
    </xacro:macro>

File: jenga_robot_description/urdf/jenga_robot.urdf.xacro (robot description, xacro)
@@ -5,5 +5,5 @@
         <xacro:include filename="$(find jenga_robot_description)/urdf/turntable.urdf.xacro"/>
 	<xacro:include filename="$(find widowx_arm_description)/urdf/widowx.urdf.xacro"/>
-<!--        <xacro:include filename="$(find jenga_robot_description)/urdf/build_platform.urdf.xacro"/> -->
+        <xacro:include filename="$(find jenga_robot_description)/urdf/build_platform.urdf.xacro"/>
 <!--        <xacro:include filename="$(find jenga_robot_description)/urdf/hopper.urdf.xacro"/> -->
 	<link name="world"/>
@@ -14,8 +14,9 @@
 		<origin xyz="0.0 0.0 0.0" rpy="0.0 0.0 0.0"/>
 	</xacro:arm_turntable>
-<!--
 	<xacro:widowx_arm parent="arm_mount_link" prefix="">
 		<origin xyz="0.0 0.0 0.0" rpy="0.0 0.0 0.0"/>
 	</xacro:widowx_arm>
--->
+	<xacro:build_platform parent="frame_main_link" prefix="">
+		<origin xyz="0.0 0.0 ${0.0254*11.2}" rpy="0.0 0.0 0.0"/>
+	</xacro:build_platform>
 </robot>
