Commit message: Moveit control is working, but is buggy
The collision mesh in moveit is not scaled, I don't know what I expected.

Will have to manually scale the stl for moveit to avoid running into the frame

File: jenga_robot_description/urdf/gazebo.urdf.xacro (robot description, xacro)
@@ -3,4 +3,8 @@
   <gazebo>
     <plugin name="ros_control" filename="libgazebo_ros_control.so"/>
+    <plugin name="mimic_joint" filename="libroboticsgroup_gazebo_mimic_joint_plugin.so">
+	<joint>gripper_joint</joint>
+	<mimicJoint>gripper_prismatic_joint_2</mimicJoint>
+    </plugin>
   </gazebo>
 </robot>

File: jenga_robot_description/urdf/turntable.urdf.xacro (robot description, xacro)
@@ -40,5 +40,5 @@
          <child link="${prefix}turntable_main_link"/>
          <axis xyz="0 0 1" />
-         <limit lower="${-M_PI/2}" upper="${M_PI/2}" effort="6" velocity="1.571" />
+         <limit lower="${-M_PI}" upper="${M_PI}" effort="6" velocity="1.571" />
       </joint>
       <joint name="${prefix}arm_mount_joint" type="fixed">
