Commit message: Fix collision mesh

File: jenga_robot_description/urdf/frame.urdf.xacro (robot description, xacro)
@@ -18,5 +18,5 @@
             <origin xyz="${12*FRAME_SCALE} ${-53.5*FRAME_SCALE} 0" rpy="0 ${-90*M_PI/180.0} 0" />
             <geometry>
-               <mesh filename="package://jenga_robot_description/meshes/frame.stl"/>
+               <mesh filename="package://jenga_robot_description/meshes/frame.stl" scale="${FRAME_SCALE} ${FRAME_SCALE} ${FRAME_SCALE}"/>
             </geometry>
          </collision>
