Commit message: Basic jenga robot is working in Gazebo

File: jenga_robot_description/urdf/turntable.urdf.xacro (robot description, xacro)
@@ -23,6 +23,6 @@
          <inertial>
             <origin xyz="0 0 0" rpy="0 0 0" />
-            <mass value="1" />
-            <inertia ixx="1.0" ixy="0.0" ixz="0.0" iyy="1.0" iyz="0.0" izz="1.0" />
+            <mass value="2" />
+            <inertia ixx="0.0262969904" ixy="0.0" ixz="0.0" iyy="0.0262969904" iyz="0.0" izz="0.05225796" />
          </inertial>
       </link>
@@ -48,3 +48,13 @@
       </joint>
    </xacro:macro>
+  <transmission name="turntable_transmission">
+    <type>transmission_interface/SimpleTransmission</type>
+    <joint name="turntable_joint">
+        <hardwareInterface>hardware_interface/PositionJointInterface</hardwareInterface>
+    </joint>
+    <actuator name="turntable_motor">
+      <hardwareInterface>EffortJointInterface</hardwareInterface>
+      <mechanicalReduction>1</mechanicalReduction>
+    </actuator>
+  </transmission>
 </robot>

Commit message: Update Rviz setup, fix positioning of arm to turntable

File: jenga_robot_description/urdf/turntable.urdf.xacro (robot description, xacro)
@@ -43,5 +43,5 @@
       </joint>
       <joint name="${prefix}arm_mount_joint" type="fixed">
-         <origin xyz="${FRAME_SCALE*4.5} 0 ${FRAME_SCALE*-1.25}" rpy="0 ${M_PI} 0" />
+         <origin xyz="${FRAME_SCALE*4.5} 0 ${FRAME_SCALE*-0.625}" rpy="0 ${M_PI} 0" />
          <parent link="${prefix}turntable_main_link" />
          <child link="${prefix}arm_mount_link" />
