Commit message: Switch to bullet physics engine so that blocks can actually stack

File: jenga_robot_description/urdf/block.urdf.xacro (robot description, xacro)
@@ -26,3 +26,25 @@
          </inertial>
       </link>
+      <gazebo reference="jenga_block_link">
+	<collision><surface>
+		<bounce><threshold>100000</threshold></bounce>
+	<friction>
+	<ode>
+        	<mu>10000000</mu>
+		<mu2>10000000</mu2>
+	        <slip1>0.0</slip1>
+		<slip2>0.0</slip2>
+	</ode>
+	<bullet>
+        	<friction>10000000</friction>
+		<friction2>10000000</friction2>
+	</bullet>
+	</friction>
+	<contact>
+		<ode><kd>100</kd></ode>
+		<bullet><kp>1000000000</kp><kd>100</kd><soft_erp>0.20</soft_erp></bullet>
+	</contact>
+	</surface></collision>
+	<material>Gazebo/Yellow</material>
+      </gazebo>
 </robot>

File: jenga_robot_description/urdf/build_platform.urdf.xacro (robot description, xacro)
@@ -35,5 +35,24 @@
          <gazebo reference="${prefix}build_platform_main_link">
                 <selfCollide>true</selfCollide>
+        <collision><surface>
+                <bounce><threshold>100000</threshold></bounce>
+        <friction>
+        <ode>
+                <mu>10000000</mu>
+                <mu2>10000000</mu2>
+                <slip1>0.0</slip1>
+                <slip2>0.0</slip2>
+        </ode>
+        <bullet>
+                <friction>10000000</friction>
+                <friction2>10000000</friction2>
+        </bullet>
+        </friction>
+        <contact>
+                <ode><kd>100</kd></ode>
+                <bullet><kp>1000000000</kp><kd>100</kd><soft_erp>0.20</soft_erp></bullet>
+        </contact>
+        </surface></collision>
          </gazebo>
-   </xacro:macro>
+    </xacro:macro>
 </robot>

File: jenga_robot_description/urdf/frame.urdf.xacro (robot description, xacro)
@@ -46,4 +46,23 @@
       </joint>
 	 <gazebo reference="${prefix}frame_main_link">
+        <collision><surface>
+                <bounce><threshold>100000</threshold></bounce>
+        <friction>
+        <ode>
+                <mu>10000000</mu>
+                <mu2>10000000</mu2>
+                <slip1>0.0</slip1>
+                <slip2>0.0</slip2>
+        </ode>
+        <bullet>
+                <friction>10000000</friction>
+                <friction2>10000000</friction2>
+        </bullet>
+        </friction>
+        <contact>
+                <ode><kd>100</kd></ode>
+                <bullet><kp>1000000000</kp><kd>100</kd><soft_erp>0.20</soft_erp></bullet>
+        </contact>
+        </surface></collision>
 		<selfCollide>true</selfCollide>
 	 </gazebo>

File: jenga_robot_description/urdf/jenga_robot.urdf.xacro (robot description, xacro)
@@ -9,5 +9,5 @@
 	<link name="world"/>
 	<xacro:jenga_frame parent="world" prefix="">
-		<origin xyz="0.0 0.0 0.0" rpy="0.0 0.0 0.0"/>
+		<origin xyz="0.0 0.0 ${0.0254*0.25}" rpy="0.0 0.0 0.0"/>
 	</xacro:jenga_frame>
 	<xacro:arm_turntable parent="frame_top_link" prefix="">
