Commit message: Updated IKFast to lower arm_base_link rather than turntable

File: jenga_robot_description/urdf/jenga_robot.urdf.xacro (robot description, xacro)
@@ -11,4 +11,5 @@
 		<origin xyz="0.0 0.0 ${0.0254*0.25}" rpy="0.0 0.0 0.0"/>
 	</xacro:jenga_frame>
+<!--xyz="0.0 0.0 0.0"-->
 	<xacro:arm_turntable parent="frame_top_link" prefix="">
 		<origin xyz="0.0 0.0 0.0" rpy="0.0 0.0 0.0"/>

File: jenga_robot_description/urdf/turntable.urdf.xacro (robot description, xacro)
@@ -43,5 +43,5 @@
       </joint>
       <joint name="${prefix}arm_mount_joint" type="fixed">
-         <origin xyz="${FRAME_SCALE*4.5} 0 ${FRAME_SCALE*-0.625}" rpy="0 ${M_PI} 0" />
+         <origin xyz="${FRAME_SCALE*4.5} 0 ${FRAME_SCALE*-3.125}" rpy="0 ${M_PI} 0" />
          <parent link="${prefix}turntable_main_link" />
          <child link="${prefix}arm_mount_link" />
